Commit message: Model bugfixing

File: model2.urdf (robot description, URDF)
Before this commit: robot manipulator, 5 links, 4 joints
Links:
- link AL_tibia_link: mass 0.08176 -> 0.18426; geometry collision box size=0.082 0.01 0.01; visual box size=0.082 0.01 0.01
- link base_link: geometry collision box size=0.0 0.0 0.0; visual box size=0.0 0.0 0.0
Joints:
- joint AL_coxa_joint: origin xyz=0.125 0.06 0 rpy=0.0 0.0 0.785398163397 -> xyz=0.0 0.0 0 rpy=0.0 0.0 0.0
- joint AL_tibia_joint: origin xyz=0.082 0 0 rpy=0.0 0.0 0.0 -> xyz=0.053 0 0 rpy=0.0 0.0 0.0
