Commit message: Bugfixing

File: phantomx_exp2.urdf (robot description, URDF)
Before this commit: robot PhantomX, 7 links, 6 joints
Joints:
- joint j_c1_lf: limit lower=-2.6179939 upper=2.6179939 effort=2.8 velocity=5.6548668 -> lower=-6.3 upper=6.3 effort=2.8 velocity=5.6548668
- joint j_thigh_lf: limit lower=-2.6179939 upper=2.6179939 effort=2.8 velocity=5.6548668 -> lower=-6.3 upper=6.3 effort=2.8 velocity=5.6548668
- joint j_tibia_lf: limit lower=-2.6179939 upper=2.6179939 effort=2.8 velocity=5.6548668 -> lower=-6.3 upper=6.3 effort=2.8 velocity=5.6548668
