Commit message: Improvements in generating the linearized dynamic model

File: test.urdf (robot description, URDF)
Before this commit: robot lbr_iiwa, 4 links, 3 joints
Joints:
- joint joint3: type revolute -> fixed

Commit message: Put propagation code in own class

File: test.urdf (robot description, URDF)
Before this commit: robot lbr_iiwa, 4 links, 3 joints
Links:
- link link1: mass 5 -> 1
- link link2: mass 5 -> 1
Joints:
- joint joint1: limit lower=-3.14159265359 upper=3.14159265359 effort=20 velocity=10 -> lower=-3.14159265359 upper=3.14159265359 effort=70 velocity=20
- joint joint2: limit lower=-3.14159265359 upper=3.14159265359 effort=1 velocity=10 -> lower=-3.14159265359 upper=3.14159265359 effort=50 velocity=20
- joint joint3: limit lower=-3.14159265359 upper=3.14159265359 effort=1 velocity=20 -> lower=-3.14159265359 upper=3.14159265359 effort=20 velocity=20

Commit message: Linearize about equilibrium space

File: test.urdf (robot description, URDF)
Before this commit: robot lbr_iiwa, 4 links, 3 joints
Joints:
- joint joint3: type fixed -> revolute

Commit message: Generate cpp code of steady state sets

File: test.urdf (robot description, URDF)
Before this commit: robot lbr_iiwa, 4 links, 3 joints
Links:
- added link link3, mass 5; collision box size=1 0.15 0.15; visual box size=1 0.15 0.15
Joints:
- added joint joint4: type fixed, parent link3, child end_effector, origin xyz=1 0 0 rpy=0 0 0, axis 0 0 1, limit lower=-3.14159265359 upper=3.14159265359 effort=10 velocity=10
- joint joint1: limit lower=-3.14159265359 upper=3.14159265359 effort=70 velocity=20 -> lower=-3.14159265359 upper=3.14159265359 effort=500 velocity=200
- joint joint2: limit lower=-3.14159265359 upper=3.14159265359 effort=50 velocity=20 -> lower=-3.14159265359 upper=3.14159265359 effort=500 velocity=200
- joint joint3: child end_effector -> link3; limit lower=-3.14159265359 upper=3.14159265359 effort=20 velocity=20 -> lower=-3.14159265359 upper=3.14159265359 effort=500 velocity=200; type fixed -> revolute

Commit message: Bugfixing

File: test.urdf (robot description, URDF)
Before this commit: robot lbr_iiwa, 5 links, 4 joints
Links:
- removed link link3
Joints:
- removed joint joint4
- joint joint1: limit lower=-3.14159265359 upper=3.14159265359 effort=500 velocity=200 -> lower=-3.14159265359 upper=3.14159265359 effort=5 velocity=200
- joint joint2: limit lower=-3.14159265359 upper=3.14159265359 effort=500 velocity=200 -> lower=-3.14159265359 upper=3.14159265359 effort=5 velocity=200
- joint joint3: child link3 -> end_effector; type revolute -> fixed

Commit message: Bugfixing

File: test.urdf (robot description, URDF)
Before this commit: robot lbr_iiwa, 4 links, 3 joints
Links:
- added link link3, mass 5; collision box size=1 0.15 0.15; visual box size=1 0.15 0.15
Joints:
- added joint joint4: type fixed, parent link3, child end_effector, origin xyz=1 0 0 rpy=0 0 0, axis 0 0 1, limit lower=-3.14159265359 upper=3.14159265359 effort=10 velocity=10
- joint joint3: child end_effector -> link3; type fixed -> revolute

Commit message: Bugfixing

File: test.urdf (robot description, URDF)
Before this commit: robot lbr_iiwa, 5 links, 4 joints
Links:
- removed link link3
Joints:
- removed joint joint4
- joint joint3: child link3 -> end_effector; type revolute -> fixed
