Commit message: Bugfixing

File: lbr_iiwa/urdf/lbr_iiwa.urdf (robot description, URDF)
Before this commit: robot lbr_iiwa, 9 links, 8 joints
Links:
- link lbr_iiwa_link_0: geometry collision mesh filename=/home/hoe01h/catkin_ws/src/lbr_iiwa/lbr_iiwa_description/me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; visual mesh filename=/home/hoe01h/catkin_ws/src/lbr_iiwa/lbr_iiwa_description/me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
- link lbr_iiwa_link_1: geometry collision mesh filename=/home/hoe01h/catkin_ws/src/lbr_iiwa/lbr_iiwa_description/me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; visual mesh filename=/home/hoe01h/catkin_ws/src/lbr_iiwa/lbr_iiwa_description/me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
- link lbr_iiwa_link_2: geometry collision mesh filename=/home/hoe01h/catkin_ws/src/lbr_iiwa/lbr_iiwa_description/me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; visual mesh filename=/home/hoe01h/catkin_ws/src/lbr_iiwa/lbr_iiwa_description/me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
- link lbr_iiwa_link_3: geometry collision mesh filename=/home/hoe01h/catkin_ws/src/lbr_iiwa/lbr_iiwa_description/me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; visual mesh filename=/home/hoe01h/catkin_ws/src/lbr_iiwa/lbr_iiwa_description/me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
- link lbr_iiwa_link_4: geometry collision mesh filename=/home/hoe01h/catkin_ws/src/lbr_iiwa/lbr_iiwa_description/me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; visual mesh filename=/home/hoe01h/catkin_ws/src/lbr_iiwa/lbr_iiwa_description/me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
- link lbr_iiwa_link_5: geometry collision mesh filename=/home/hoe01h/catkin_ws/src/lbr_iiwa/lbr_iiwa_description/me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; visual mesh filename=/home/hoe01h/catkin_ws/src/lbr_iiwa/lbr_iiwa_description/me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
- link lbr_iiwa_link_6: geometry collision mesh filename=/home/hoe01h/catkin_ws/src/lbr_iiwa/lbr_iiwa_description/me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; visual mesh filename=/home/hoe01h/catkin_ws/src/lbr_iiwa/lbr_iiwa_description/me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
- link lbr_iiwa_link_7: geometry collision mesh filename=/home/hoe01h/catkin_ws/src/lbr_iiwa/lbr_iiwa_description/me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; visual mesh filename=/home/hoe01h/catkin_ws/src/lbr_iiwa/lbr_iiwa_description/me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
