Commit message: Included meshfree lbr iiwa model + urdf loader

File: lbr_iiwa/urdf/lbr_iiwa_meshfree.urdf (robot description, URDF)
Before this commit: robot lbr_iiwa, 9 links, 8 joints
Links:
- link lbr_iiwa_link_0: geometry collision box size=0.15 0.15 0.1575; visual box size=0.15 0.15 0.1575
- link lbr_iiwa_link_1: geometry collision box size=0.05 0.05 0.2025; visual box size=0.05 0.05 0.2025
- link lbr_iiwa_link_2: geometry collision box size=0.05 0.2045 0.05; visual box size=0.05 0.2045 0.05
- link lbr_iiwa_link_3: geometry collision box size=0.05 0.05 0.2155; visual box size=0.05 0.05 0.2155
- link lbr_iiwa_link_4: geometry collision box size=0.05 0.1845 0.05; visual box size=0.05 0.1845 0.05
- link lbr_iiwa_link_5: geometry collision box size=0.05 0.05 0.2155; visual box size=0.05 0.05 0.2155
- link lbr_iiwa_link_6: geometry collision box size=0.05 0.081 0.05; visual box size=0.05 0.081 0.05
- link lbr_iiwa_link_7: geometry collision box size=0.05 0.05 0.04; visual box size=0.05 0.05 0.04

Commit message: Successfully integrated simulation environment

File: lbr_iiwa/urdf/lbr_iiwa_meshfree.urdf (robot description, URDF)
Before this commit: robot lbr_iiwa, 9 links, 8 joints
Links:
- removed link lbr_iiwa_link_4
- removed link lbr_iiwa_link_5
- removed link lbr_iiwa_link_6
- removed link lbr_iiwa_link_7
Joints:
- removed joint lbr_iiwa_joint_4
- removed joint lbr_iiwa_joint_5
- removed joint lbr_iiwa_joint_6
- removed joint lbr_iiwa_joint_7
- joint lbr_iiwa_joint_1: limit lower=-2.96705972839 upper=2.96705972839 effort=300 velocity=10 -> lower=-3.14159265359 upper=3.14159265359 effort=300 velocity=10
- joint lbr_iiwa_joint_3: axis 0 0 1 -> 0 1 0
- joint world_joint: origin xyz=0 0 0.0 rpy=0 0 0 -> xyz=0 0 0.0 rpy=-1 0 0

File: lbr_iiwa/urdf/lbr_iiwa_meshfree.urdf.xacro (robot description, xacro)
@@ -2,7 +2,7 @@
 <robot name="lbr_iiwa" xmlns:xacro="http://www.ros.org/wiki/xacro">
   <!-- Import Rviz colors -->
-  <xacro:include filename="$(find lbr_iiwa_description)/urdf/materials.xacro" />
+  <xacro:include filename="materials.xacro" />
   <!--Import the lbr iiwa macro -->
-  <xacro:include filename="$(find lbr_iiwa_description)/urdf/lbr_iiwa_meshfree.xacro"/>
+  <xacro:include filename="lbr_iiwa_meshfree_simple.xacro"/>
  <!-- Import Gazebo plugins -->
   <xacro:include filename="$(find lbr_iiwa_description)/gazebo/gazebo.urdf.xacro"/>
@@ -11,5 +11,5 @@
   <!--lbr-->
   <xacro:lbr_iiwa name="lbr_iiwa" hardware_interface="$(arg prefix)" parent="world">
-    <origin xyz="0 0 0.0" rpy="0 0 0" />
+    <origin xyz="0 0 0.0" rpy="-1 0 0" />
   </xacro:lbr_iiwa>
 </robot>

File: lbr_iiwa/urdf/lbr_iiwa_meshfree_simple.xacro (robot description, xacro)
@@ -130,5 +130,5 @@
       <child link="${name}_link_3"/>
       <origin xyz="0 0.2045 0" rpy="${PI / 2} 0 ${PI}"/>
-      <axis xyz="0 0 1"/>
+      <axis xyz="0 1 0"/>
       <limit lower="${-170 * PI / 180}" upper="${170 * PI / 180}"
              effort="${max_effort}" velocity="${max_velocity}" />
@@ -160,144 +160,4 @@
       </collision>
     </link>
-   <!-- joint between link_3 and link_4 -->
-    <joint name="${name}_joint_4" type="revolute">
-      <parent link="${name}_link_3"/>
-      <child link="${name}_link_4"/>
-      <origin xyz="0 0 0.2155" rpy="${PI / 2} 0 0"/>
-      <axis xyz="0 0 1"/>
-      <limit lower="${-120 * PI / 180}" upper="${120 * PI / 180}"
-             effort="${max_effort}" velocity="${max_velocity}" />
-      <!-- <safety_controller soft_lower_limit="${-118 * PI / 180}"
-           soft_upper_limit="${118 * PI / 180}"
-           k_position="${safety_controller_k_pos}"
-           k_velocity="${safety_controller_k_vel}"/> -->
-      <dynamics damping="${joint_damping}"/>
-    </joint>
-    <link name="${name}_link_4">
-      <inertial>
-        <origin xyz="0 0.067 0.034" rpy="0 0 0"/>
-        <mass value="2.7"/>
-        <inertia ixx="0.03"  ixy="0"  ixz="0" iyy="0.01" iyz="0" izz="0.029" />
-      </inertial>
-      <visual>
-        <origin xyz="0 ${len_link_4 / 2} 0" rpy="0 0 0"/>
-        <geometry>
-          <box size="0.05 ${len_link_4} 0.05"/>
-        </geometry>
-        <material name="Orange"/>
-      </visual>
-      <collision>
-        <origin xyz="0 ${len_link_4 / 2} 0" rpy="0 0 0"/>
-        <geometry>
-          <box size="0.05 ${len_link_4} 0.05"/>
-        </geometry>
-        <material name="Orange"/>
-      </collision>
-    </link>
-    <!-- joint between link_4 and link_5 -->
-    <joint name="${name}_joint_5" type="revolute">
-      <parent link="${name}_link_4"/>
-      <child link="${name}_link_5"/>
-      <origin xyz="0 0.1845 0" rpy="${-PI / 2} ${PI} 0"/>
-      <axis xyz="0 0 1"/>
-      <limit lower="${-170 * PI / 180}" upper="${170 * PI / 180}"
-             effort="${max_effort}" velocity="${max_velocity}" />
-      <!-- <safety_controller soft_lower_limit="${-118 * PI / 180}"
-           soft_upper_limit="${118 * PI / 180}"
-           k_position="${safety_controller_k_pos}"
-           k_velocity="${safety_controller_k_vel}"/> -->
-      <dynamics damping="${joint_damping}"/>
-    </joint>
-    <link name="${name}_link_5">
-      <inertial>
-        <origin xyz="0.0001 0.021 0.076" rpy="0 0 0"/>
-        <mass value="1.7"/>
-        <inertia ixx="0.02"  ixy="0"  ixz="0" iyy="0.018" iyz="0" izz="0.005" />
-      </inertial>
-      <visual>
-        <origin xyz="0 0 ${len_link_5 / 2}" rpy="0 0 0"/>
-        <geometry>
-          <box size="0.05 0.05 ${len_link_5}"/>
-        </geometry>
-        <material name="Orange"/>
-      </visual>
-      <collision>
-        <origin xyz="0 0 ${len_link_5 / 2}" rpy="0 0 0"/>
-        <geometry>
-          <box size="0.05 0.05 ${len_link_5}"/>
-        </geometry>
-        <material name="Orange"/>
-      </collision>
-    </link>
- <!-- joint between link_5 and link_6 -->
-    <joint name="${name}_joint_6" type="revolute">
-      <parent link="${name}_link_5"/>
-      <child link="${name}_link_6"/>
-      <origin xyz="0 0 0.2155" rpy="${PI / 2} 0 0"/>
-      <axis xyz="0 0 1"/>
-      <limit lower="${-120 * PI / 180}" upper="${120 * PI / 180}"
-             effort="${max_effort}" velocity="${max_velocity}" />
-      <!-- <safety_controller soft_lower_limit="${-118 * PI / 180}"
-           soft_upper_limit="${118 * PI / 180}"
-           k_position="${safety_controller_k_pos}"
-           k_velocity="${safety_controller_k_vel}"/> -->
-      <dynamics damping="${joint_damping}"/>
-    </joint>
-    <link name="${name}_link_6">
-      <inertial>
-        <origin xyz="0 0.0006 0.0004" rpy="0 0 0"/>
-        <mass value="1.8"/>
-        <inertia ixx="0.005"  ixy="0"  ixz="0" iyy="0.0036" iyz="0" izz="0.0047" />
-      </inertial>
-      <visual>
-        <origin xyz="0 ${len_link_6 / 2} 0" rpy="0 0 0"/>
-        <geometry>
-          <box size="0.05 ${len_link_6} 0.05"/>
-        </geometry>
-        <material name="Orange"/>
-      </visual>
-      <collision>
-        <origin xyz="0 ${len_link_6 / 2} 0" rpy="0 0 0"/>
-        <geometry>
-          <box size="0.05 ${len_link_6} 0.05"/>
-        </geometry>
-        <material name="Orange"/>
-      </collision>
-    </link>
- <!-- joint between link_6 and link_7 -->
-    <joint name="${name}_joint_7" type="revolute">
-      <parent link="${name}_link_6"/>
-      <child link="${name}_link_7"/>
-      <origin xyz="0 0.081 0" rpy="${- PI / 2} ${PI} 0"/>
-      <axis xyz="0 0 1"/>
-      <limit lower="${-190 * PI / 180}" upper="${190 * PI / 180}"
-             effort="${max_effort}" velocity="${max_velocity}" />
-      <!-- <safety_controller soft_lower_limit="${-118 * PI / 180}"
-           soft_upper_limit="${118 * PI / 180}"
-           k_position="${safety_controller_k_pos}"
-           k_velocity="${safety_controller_k_vel}"/> -->
-      <dynamics damping="${joint_damping}"/>
-    </joint>
-    <link name="${name}_link_7">
-      <inertial>
-        <origin xyz="0 0 0.02" rpy="0 0 0"/>
-        <mass value="0.3"/>
-        <inertia ixx="0.001"  ixy="0"  ixz="0" iyy="0.001" iyz="0" izz="0.001" />
-      </inertial>
-      <visual>
-        <origin xyz="0 0 ${len_link_7 / 2}" rpy="0 0 0"/>
-        <geometry>
-          <box size="0.05 0.05 ${len_link_7}"/>
-        </geometry>
-        <material name="Grey"/>
-      </visual>
-      <collision>
-        <origin xyz="0 0 ${len_link_7 / 2}" rpy="0 0 0"/>
-        <geometry>
-          <box size="0.05 0.05 ${len_link_7}"/>
-        </geometry>
-        <material name="Grey"/>
-      </collision>
-    </link>
     <!--Extensions -->
     <xacro:lbr_iiwa_gazebo name="${name}" />

File: phantomx_exp2.urdf (robot description, URDF)
Before this commit: robot PhantomX, 7 links, 6 joints
Links:
- removed link base_link
- link c1_lf: geometry collision box size=0.045 0.022 0.0325; visual box size=0.045 0.054 0.0325
- link c2_lf: geometry collision box size=0.045 0.022 0.0325; visual box size=0.0645 0.022 0.0325
- link tibia_lf: geometry collision box size=0.045 0.022 0.0325; visual box size=0.0645 0.022 0.325
Joints:
- removed joint j_phantomx_attachment
- joint world_base_link: axis 0 0 1 -> (none); child base_link -> MP_BODY

Commit message: RRT working now

File: lbr_iiwa/urdf/lbr_iiwa_meshfree.urdf (robot description, URDF)
Before this commit: robot lbr_iiwa, 5 links, 4 joints
Joints:
- joint lbr_iiwa_joint_1: limit lower=-3.14159265359 upper=3.14159265359 effort=300 velocity=10 -> lower=-3.14159265359 upper=3.14159265359 effort=300 velocity=30
- joint lbr_iiwa_joint_2: limit lower=-2.09439510239 upper=2.09439510239 effort=300 velocity=10 -> lower=-2.09439510239 upper=2.09439510239 effort=300 velocity=30
- joint lbr_iiwa_joint_3: limit lower=-2.96705972839 upper=2.96705972839 effort=300 velocity=10 -> lower=-2.96705972839 upper=2.96705972839 effort=300 velocity=30

File: lbr_iiwa/urdf/lbr_iiwa_meshfree_simple.xacro (robot description, xacro)
@@ -12,5 +12,5 @@
   <xacro:property name="joint_damping" value="0.5" />
   <xacro:property name="max_effort" value="300"/>
-  <xacro:property name="max_velocity" value="10"/>
+  <xacro:property name="max_velocity" value="30"/>
   <xacro:property name="len_link_0" value="0.1575"/>
   <xacro:property name="len_link_1" value="0.2025"/>

Commit message: Bugfixing

File: lbr_iiwa/urdf/lbr_iiwa_meshfree.urdf (robot description, URDF)
Before this commit: robot lbr_iiwa, 5 links, 4 joints
Joints:
- joint world_joint: origin xyz=0 0 0.0 rpy=-1 0 0 -> xyz=0 0 0.0 rpy=0 0 0

File: lbr_iiwa/urdf/lbr_iiwa_meshfree.urdf.xacro (robot description, xacro)
@@ -11,5 +11,5 @@
   <!--lbr-->
   <xacro:lbr_iiwa name="lbr_iiwa" hardware_interface="$(arg prefix)" parent="world">
-    <origin xyz="0 0 0.0" rpy="-1 0 0" />
+    <origin xyz="0 0 0.0" rpy="0 0 0" />
   </xacro:lbr_iiwa>
 </robot>

Commit message: Parameter tuning

File: lbr_iiwa/urdf/lbr_iiwa_meshfree.urdf (robot description, URDF)
Before this commit: robot lbr_iiwa, 5 links, 4 joints
Joints:
- joint lbr_iiwa_joint_1: limit lower=-3.14159265359 upper=3.14159265359 effort=300 velocity=30 -> lower=-3.14159265359 upper=3.14159265359 effort=10 velocity=50
- joint lbr_iiwa_joint_2: limit lower=-2.09439510239 upper=2.09439510239 effort=300 velocity=30 -> lower=-2.09439510239 upper=2.09439510239 effort=20 velocity=50
- joint lbr_iiwa_joint_3: limit lower=-2.96705972839 upper=2.96705972839 effort=300 velocity=30 -> lower=-2.96705972839 upper=2.96705972839 effort=20 velocity=50
- joint world_joint: origin xyz=0 0 0.0 rpy=0 0 0 -> xyz=0 0 0.0 rpy=3.14 0 0

File: lbr_iiwa/urdf/lbr_iiwa_meshfree.urdf.xacro (robot description, xacro)
@@ -11,5 +11,5 @@
   <!--lbr-->
   <xacro:lbr_iiwa name="lbr_iiwa" hardware_interface="$(arg prefix)" parent="world">
-    <origin xyz="0 0 0.0" rpy="0 0 0" />
+    <origin xyz="0 0 0.0" rpy="3.14 0 0" />
   </xacro:lbr_iiwa>
 </robot>

File: lbr_iiwa/urdf/lbr_iiwa_meshfree_simple.xacro (robot description, xacro)
@@ -11,6 +11,8 @@
   <xacro:property name="safety_controller_k_vel" value="2" /> -->
   <xacro:property name="joint_damping" value="0.5" />
-  <xacro:property name="max_effort" value="300"/>
-  <xacro:property name="max_velocity" value="30"/>
+  <xacro:property name="max_effort_joint1" value="10"/>
+  <xacro:property name="max_effort_joint2" value="30"/>
+  <xacro:property name="max_effort_joint3" value="30"/>
+  <xacro:property name="max_velocity" value="50"/>
   <xacro:property name="len_link_0" value="0.1575"/>
   <xacro:property name="len_link_1" value="0.2025"/>
@@ -62,5 +64,5 @@
       <axis xyz="0 0 1"/>
       <limit lower="${-180 * PI / 180}" upper="${180 * PI / 180}"
-             effort="${max_effort}" velocity="${max_velocity}" />
+             effort="${max_effort_joint1}" velocity="${max_velocity}" />
       <!--   <safety_controller soft_lower_limit="${-168 * M_PI / 180}"
            soft_upper_limit="${168 * M_PI / 180}"
@@ -97,5 +99,5 @@
       <axis xyz="0 0 1"/>
       <limit lower="${-120 * PI / 180}" upper="${120 * PI / 180}"
-             effort="${max_effort}" velocity="${max_velocity}" />
+             effort="${max_effort_joint2}" velocity="${max_velocity}" />
       <!-- <safety_controller soft_lower_limit="${-118 * PI / 180}"
            soft_upper_limit="${118 * PI / 180}"
@@ -132,5 +134,7 @@
       <axis xyz="0 1 0"/>
       <limit lower="${-170 * PI / 180}" upper="${170 * PI / 180}"
-             effort="${max_effort}" velocity="${max_velocity}" />
+             effort="${max_effort_joint3}" velocity="${max_velocity}" />
+      <!--limit lower="0" upper="0"
+             effort="${max_effort_joint3}" velocity="${max_velocity}" /-->
       <!-- <safety_controller soft_lower_limit="${-118 * PI / 180}"
            soft_upper_limit="${118 * PI / 180}"

Commit message: Added symbolic model generator

File: lbr_iiwa/urdf/lbr_iiwa_meshfree.urdf (robot description, URDF)
Before this commit: robot lbr_iiwa, 5 links, 4 joints
Joints:
- joint lbr_iiwa_joint_1: limit lower=-3.14159265359 upper=3.14159265359 effort=10 velocity=50 -> lower=-3.14159265359 upper=3.14159265359 effort=10 velocity=10
- joint lbr_iiwa_joint_2: limit lower=-2.09439510239 upper=2.09439510239 effort=20 velocity=50 -> lower=-2.09439510239 upper=2.09439510239 effort=20 velocity=10
- joint lbr_iiwa_joint_3: limit lower=-2.96705972839 upper=2.96705972839 effort=20 velocity=50 -> lower=-2.96705972839 upper=2.96705972839 effort=10 velocity=10

File: lbr_iiwa/urdf/lbr_iiwa_meshfree_simple.xacro (robot description, xacro)
@@ -12,7 +12,7 @@
   <xacro:property name="joint_damping" value="0.5" />
   <xacro:property name="max_effort_joint1" value="10"/>
-  <xacro:property name="max_effort_joint2" value="30"/>
-  <xacro:property name="max_effort_joint3" value="30"/>
-  <xacro:property name="max_velocity" value="50"/>
+  <xacro:property name="max_effort_joint2" value="20"/>
+  <xacro:property name="max_effort_joint3" value="10"/>
+  <xacro:property name="max_velocity" value="10"/>
   <xacro:property name="len_link_0" value="0.1575"/>
   <xacro:property name="len_link_1" value="0.2025"/>
